File: statie_lipit/development/hardware/control.sch (EAGLE design)
At the start: 13 parts, among them IC1 MEGA8-AI, J1 22-05-7038-03, J2 con)ach, J3 22-05-7038-03, J4 22-05-7088-08

Commit message: new hardware design
Parts:
- added TP1, TP2, TP3, TP4, TP5, TP6: TPSQPAD1-13, testpad:TPSQPAD1-13
Connections:
- removed net LINE2: IC1.PB2(SS/OC1B), J2-6.S
- removed net LINE3: IC1.PB5(SCK), J2-7.S, J4-6.S
- removed net LINE4: IC1.PB3(MOSI/OC2), IC1.PC0(ADC0), J2-8.S, J4-7.S
- removed net LINE5: IC1.PB0(ICP), J4-8.S
- new net D/C: IC1.PB7(XTAL2/TOSC2)
- new net MISO: IC1.PB4(MISO), J2-7.S, TP1.TP
- new net MOSI: IC1.PB3(MOSI/OC2), J4-7.S, TP4.TP
- new net RES: IC1.PB6(XTAL1/TOSC1)
- new net RST: IC1.PC6(/RESET), TP5.TP
- new net SCK: IC1.PB5(SCK), J2-6.S, J4-8.S, TP3.TP
- new net SS_1: IC1.PB2(SS/OC1B), J2-8.S
- new net SS_2: IC1.PB0(ICP), J4-6.S
- net 5V_LOGIC: now also TP2.TP
- net BUT1: now also IC1.PD5(T1); no longer IC1.PD2(INT0)
- net BUT2: now also IC1.PD6(AIN0); no longer IC1.PD3(INT1)
- net BUT3: now also IC1.PD7(AIN1); no longer IC1.PD4(XCK/T0)
- net GND: now also TP6.TP
- net ID1: now also IC1.PC2(ADC2); no longer IC1.PD5(T1)
- net ID2: now also IC1.PC1(ADC1); no longer IC1.PD6(AIN0)
- net LINE1: now also IC1.PC0(ADC0); no longer IC1.PB4(MISO)
